Commit message: regen urdf with correct paths

File: moveit_config/config/ur.urdf (robot description, URDF)
Before this commit: robot ur, 34 links, 33 joints
Links:
- link camera_head_link: geometry collision box size=0.02505 0.09 0.025; visual mesh filename=file:///home/asimov/UR3_ROS2_PICK_AND_PLACE/install/ur_desc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
- link robotiq_arg2f_base_link: geometry collision mesh filename=package://robotiq_2f_85_gripper_visualization/meshes/collis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; visual mesh filename=package://robotiq_2f_85_gripper_visualization/meshes/collis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
Joints:
- joint wrist_3_joint: limit effort=12.0 velocity=6.283185307179586 -> lower=-6.283185307179586 upper=6.283185307179586 effort=12.0 velocity=6.283185307179586; type continuous -> revolute

Commit message: camera tilt 70deg, cylinders 15cm tall in world

File: moveit_config/config/ur.urdf (robot description, URDF)
Before this commit: robot ur, 34 links, 33 joints
Joints:
- joint camera_head_joint: origin xyz=0 0.01 0.70 rpy=0.0 0.4363323129985824 1.5707963267948966 -> xyz=0 0.01 0.70 rpy=0.0 1.2217304763960306 1.5707963267948966

File: ur_description/urdf/intel_rgbd_cam_d435.urdf.xacro (robot description, xacro)
@@ -12,5 +12,5 @@
     <xacro:property name="d435_cam_depth_to_infra2_offset" value="-0.050"/>
     <xacro:property name="d435_cam_depth_to_color_offset" value="0.015"/>
-    <xacro:property name="camera_tilt_angle_deg" value="55"/>
+    <xacro:property name="camera_tilt_angle_deg" value="70"/>
   <link name="torso_link">
   <inertial>

Commit message: restore camera 25deg z=0.50; fix point cloud TF frame to depth_optical; fix pick_and_place_demo.world

File: moveit_config/config/ur.urdf (robot description, URDF)
Before this commit: robot ur, 34 links, 33 joints
Joints:
- joint camera_head_joint: origin xyz=0 0.01 0.70 rpy=0.0 1.2217304763960306 1.5707963267948966 -> xyz=0 0.01 0.50 rpy=0.0 0.4363323129985824 1.5707963267948966

File: ur_description/urdf/intel_rgbd_cam_d435.urdf.xacro (robot description, xacro)
@@ -12,5 +12,5 @@
     <xacro:property name="d435_cam_depth_to_infra2_offset" value="-0.050"/>
     <xacro:property name="d435_cam_depth_to_color_offset" value="0.015"/>
-    <xacro:property name="camera_tilt_angle_deg" value="70"/>
+    <xacro:property name="camera_tilt_angle_deg" value="25"/>
   <link name="torso_link">
   <inertial>
@@ -58,5 +58,5 @@
       <parent link="torso_link"/>
       <child link="camera_head_link" />
-      <origin xyz="0 0.01 0.70" rpy="0.0 ${camera_tilt_angle_deg * M_PI / 180} ${M_PI/2}"/>
+      <origin xyz="0 0.01 0.50" rpy="0.0 ${camera_tilt_angle_deg * M_PI / 180} ${M_PI/2}"/>
     </joint>
     <link name="camera_head_link">
@@ -145,5 +145,8 @@
     <always_on>1</always_on>
     <update_rate>10</update_rate>
-    <gz_frame_id>camera_head_link</gz_frame_id>
+    <!-- Use depth optical frame: Ignition outputs point cloud in Z-forward optical
+         convention, so the frame_id must match the optical frame (not camera_head_link
+         which has a different orientation from the mounting joint RPY). -->
+    <gz_frame_id>camera_head_depth_optical_frame</gz_frame_id>
     <visualize>true</visualize>
   </sensor>

Commit message: fix point cloud viewer: camera at stick top (z=0.70), add left_outer_knuckle initial pos, remove PlanningScene from point_cloud.rviz, update README

File: moveit_config/config/ur.urdf (robot description, URDF)
Before this commit: robot ur, 34 links, 33 joints
Joints:
- joint camera_head_joint: origin xyz=0 0.01 0.50 rpy=0.0 0.4363323129985824 1.5707963267948966 -> xyz=0 0.01 0.70 rpy=0.0 0.4363323129985824 1.5707963267948966

File: ur_description/urdf/intel_rgbd_cam_d435.urdf.xacro (robot description, xacro)
@@ -58,5 +58,5 @@
       <parent link="torso_link"/>
       <child link="camera_head_link" />
-      <origin xyz="0 0.01 0.50" rpy="0.0 ${camera_tilt_angle_deg * M_PI / 180} ${M_PI/2}"/>
+      <origin xyz="0 0.01 0.70" rpy="0.0 ${camera_tilt_angle_deg * M_PI / 180} ${M_PI/2}"/>
     </joint>
     <link name="camera_head_link">

Commit message: fix point cloud QoS, camera at 0.50m, fix crop bounds for segmentation, update CONCEPTS.md and README

File: moveit_config/config/ur.urdf (robot description, URDF)
Before this commit: robot ur, 34 links, 33 joints
Joints:
- joint camera_head_joint: origin xyz=0 0.01 0.70 rpy=0.0 0.4363323129985824 1.5707963267948966 -> xyz=0 0.01 0.50 rpy=0.0 0.4363323129985824 1.5707963267948966

File: ur_description/urdf/intel_rgbd_cam_d435.urdf.xacro (robot description, xacro)
@@ -58,5 +58,5 @@
       <parent link="torso_link"/>
       <child link="camera_head_link" />
-      <origin xyz="0 0.01 0.70" rpy="0.0 ${camera_tilt_angle_deg * M_PI / 180} ${M_PI/2}"/>
+      <origin xyz="0 0.01 0.50" rpy="0.0 ${camera_tilt_angle_deg * M_PI / 180} ${M_PI/2}"/>
     </joint>
     <link name="camera_head_link">
