Commit message: add gripper launch arg

File: moveit_config/config/ur.urdf.xacro (robot description, xacro)
@@ -2,17 +2,44 @@
 <robot xmlns:xacro="http://www.ros.org/wiki/xacro" name="ur">
     <xacro:arg name="initial_positions_file" default="initial_positions.yaml" />
-   <xacro:arg name="use_gazebo" default="true"/> <!-- Added missing argument -->
-   <xacro:arg name="robot_name" default="ur"/>
-    <!-- Import ur urdf file -->
-    <xacro:include filename="$(find ur_description)/urdf/ur.urdf.xacro" />
-    <!-- Import control_xacro -->
+    <xacro:arg name="use_gazebo" default="true"/> <!-- Added missing argument -->
+    <xacro:arg name="robot_name" default="ur"/>
+    <xacro:arg name="gripper" default="robotiq_2f_85"/>
+    <xacro:arg name="name" default="ur"/>
+    <xacro:arg name="ur_type" default="ur3"/>
+    <xacro:arg name="tf_prefix" default=""/>
+    <xacro:arg name="joint_limit_params" default="$(find ur_description)/config/$(arg ur_type)/joint_limits.yaml"/>
+    <xacro:arg name="kinematics_params" default="$(find ur_description)/config/$(arg ur_type)/default_kinematics.yaml"/>
+    <xacro:arg name="physical_params" default="$(find ur_description)/config/$(arg ur_type)/physical_parameters.yaml"/>
+    <xacro:arg name="visual_params" default="$(find ur_description)/config/$(arg ur_type)/visual_parameters.yaml"/>
+    <xacro:arg name="safety_limits" default="false"/>
+    <xacro:arg name="safety_pos_margin" default="0.15"/>
+    <xacro:arg name="safety_k_position" default="20"/>
+    <xacro:arg name="force_abs_paths" default="false"/>
+    <xacro:include filename="$(find ur_description)/urdf/ur_macro.xacro" />
     <xacro:include filename="$(find moveit_config)/config/ur.ros2_control.xacro" />
+    <xacro:include filename="$(find ur_description)/urdf/gazebo_sim_ros2_control.urdf.xacro" />
+    <link name="world" />
+    <xacro:ur_robot
+      name="$(arg name)"
+      tf_prefix="$(arg tf_prefix)"
+      parent="world"
+      joint_limits_parameters_file="$(arg joint_limit_params)"
+      kinematics_parameters_file="$(arg kinematics_params)"
+      physical_parameters_file="$(arg physical_params)"
+      visual_parameters_file="$(arg visual_params)"
+      safety_limits="$(arg safety_limits)"
+      safety_pos_margin="$(arg safety_pos_margin)"
+      safety_k_position="$(arg safety_k_position)"
+      force_abs_paths="$(arg force_abs_paths)"
+      gripper="$(arg gripper)">
+      <origin xyz="0 0 0" rpy="0 0 0" />
+    </xacro:ur_robot>
     <gazebo>
-  <disableFixedJointLumping>true</disableFixedJointLumping>
-</gazebo>
+      <disableFixedJointLumping>true</disableFixedJointLumping>
+    </gazebo>
     <xacro:ur_ros2_control name="ur" initial_positions_file="$(find moveit_config)/config/initial_positions.yaml"/>
-    <xacro:include filename="$(find ur_description)/urdf/gazebo_sim_ros2_control.urdf.xacro" />
-   <xacro:load_gazebo_sim_ros2_control_plugin
-     robot_name="$(arg robot_name)"
-     use_gazebo="$(arg use_gazebo)"/>
+    <xacro:load_gazebo_sim_ros2_control_plugin
+      robot_name="$(arg robot_name)"
+      use_gazebo="$(arg use_gazebo)"/>
+    <xacro:include filename="$(find ur_description)/urdf/intel_rgbd_cam_d435.urdf.xacro"/>
 </robot>

File: ur_description/urdf/ur_macro.xacro (robot description, xacro)
@@ -2,5 +2,7 @@
 <robot xmlns:xacro="http://wiki.ros.org/xacro">
   <xacro:include filename="$(find ur_description)/urdf/inc/ur_common.xacro" />
-   <xacro:include filename="$(find robotiq_2f_85_gripper_visualization)/urdf/robotiq_arg2f_85_model_macro.xacro"/>
+  <xacro:include filename="$(find robotiq_2f_85_gripper_visualization)/urdf/robotiq_arg2f_85_model_macro.xacro"/>
+  <xacro:include filename="$(find robotiq_description)/urdf/robotiq_2f_140_macro.urdf.xacro"/>
+  <xacro:include filename="$(find onrobot_description)/urdf/onrobot_rg.urdf.xacro"/>
   <xacro:macro name="ur_robot" params="
     name
@@ -16,4 +18,5 @@
     safety_k_position:=20
     force_abs_paths:=false
+    gripper:=robotiq_2f_85
     ">
     <!-- Load configuration data from the provided .yaml files -->
@@ -334,18 +337,32 @@
   <child link="${tf_prefix}tool0"/>
   </joint>
-   <xacro:include filename="$(find robotiq_2f_85_gripper_visualization)/urdf/robotiq_arg2f_85_model_macro.xacro"/>
-  <!-- Include the gripper Xacro file  -->
-<xacro:robotiq_arg2f_85 prefix=""/>
-<!-- Attach the gripper to tool0 -->
-<!-- Attach gripper to wrist_3_link with corrected rotation -->
-<joint name="${tf_prefix}gripper_joint" type="fixed">
-  <parent link="${tf_prefix}tool0"/>
-  <child link="${tf_prefix}robotiq_arg2f_base_link"/>
-  <origin xyz="0 0 0.005" rpy="0 0 0"/>
-    <gazebo>
-    <disableFixedJointLumping>true</disableFixedJointLumping>
-  </gazebo>
-</joint>
-<!-- Define the gripper with a meaningful prefix -->
+  <!-- Robotiq 2F-85 -->
+  <xacro:if value="${gripper == 'robotiq_2f_85'}">
+    <xacro:robotiq_arg2f_85 prefix=""/>
+    <joint name="${tf_prefix}gripper_joint" type="fixed">
+      <parent link="${tf_prefix}tool0"/>
+      <child link="${tf_prefix}robotiq_arg2f_base_link"/>
+      <origin xyz="0 0 0.005" rpy="0 0 0"/>
+      <gazebo><disableFixedJointLumping>true</disableFixedJointLumping></gazebo>
+    </joint>
+  </xacro:if>
+  <!-- Robotiq 2F-140 -->
+  <xacro:if value="${gripper == 'robotiq_2f_140'}">
+    <xacro:robotiq_gripper name="robotiq_140" prefix="" parent="${tf_prefix}tool0" include_ros2_control="false">
+      <origin xyz="0 0 0.005" rpy="0 0 0"/>
+    </xacro:robotiq_gripper>
+  </xacro:if>
+  <!-- OnRobot RG2 -->
+  <xacro:if value="${gripper == 'onrobot_rg2'}">
+    <xacro:onrobot_rg prefix="" model="rg2_v1" parent="${tf_prefix}tool0" standalone="false">
+      <origin xyz="0 0 0.01" rpy="0 0 ${pi/2}"/>
+    </xacro:onrobot_rg>
+  </xacro:if>
+  <!-- OnRobot RG6 -->
+  <xacro:if value="${gripper == 'onrobot_rg6'}">
+    <xacro:onrobot_rg prefix="" model="rg6_v1" parent="${tf_prefix}tool0" standalone="false">
+      <origin xyz="0 0 0.01" rpy="0 0 ${pi/2}"/>
+    </xacro:onrobot_rg>
+  </xacro:if>
   </xacro:macro>
 </robot>
