Commit message: add mount table to world

File: moveit_config/config/ur.urdf.xacro (robot description, xacro)
@@ -16,4 +16,5 @@
     <xacro:arg name="safety_k_position" default="20"/>
     <xacro:arg name="force_abs_paths" default="false"/>
+    <xacro:arg name="table_height" default="0.0"/>
     <xacro:include filename="$(find ur_description)/urdf/ur_macro.xacro" />
     <xacro:include filename="$(find moveit_config)/config/ur.ros2_control.xacro" />
@@ -38,5 +39,5 @@
       force_abs_paths="$(arg force_abs_paths)"
       gripper="$(arg gripper)">
-      <origin xyz="0 0 0" rpy="0 0 0" />
+      <origin xyz="0 0 $(arg table_height)" rpy="0 0 0" />
     </xacro:ur_robot>
     <gazebo>

File: ur_description/urdf/intel_rgbd_cam_d435.urdf.xacro (robot description, xacro)
@@ -12,5 +12,5 @@
     <xacro:property name="d435_cam_depth_to_infra2_offset" value="-0.050"/>
     <xacro:property name="d435_cam_depth_to_color_offset" value="0.015"/>
-    <xacro:property name="camera_tilt_angle_deg" value="25"/>
+    <xacro:property name="camera_tilt_angle_deg" value="55"/>
   <link name="torso_link">
   <inertial>
