Commit message: gripper mimic joint init: add per-joint keys, add missing left_outer_knuckle; update BUGS_FIXED

File: moveit_config/config/ur.ros2_control.xacro (robot description, xacro)
@@ -78,13 +78,26 @@
                 </state_interface>
             </joint>
-            <!-- Mimic joints (no command interfaces, initial value same as finger_joint) -->
+            <!-- Mimic joints (no command interfaces, each with explicit initial_value key
+                 so Ignition Gazebo initialises every joint individually rather than
+                 sharing the finger_joint reference which caused right-side joints to
+                 start at their limit positions). -->
+            <!-- left_outer_knuckle_joint (was missing — added) -->
+            <joint name="left_outer_knuckle_joint">
+                <state_interface name="position">
+                    <param name="initial_value">${initial_positions['left_outer_knuckle_joint']}</param>
+                </state_interface>
+                <state_interface name="velocity"/>
+                <state_interface name="effort">
+                    <param name="effort_limit">100.0</param>
+                </state_interface>
+            </joint>
             <!-- right_outer_knuckle_joint -->
             <joint name="right_outer_knuckle_joint">
                 <state_interface name="position">
-                    <param name="initial_value">${initial_positions['finger_joint']}</param>
+                    <param name="initial_value">${initial_positions['right_outer_knuckle_joint']}</param>
                 </state_interface>
                 <state_interface name="velocity"/>
                 <state_interface name="effort">
-                    <param name="effort_limit">100.0</param> <!-- Increased effort for knuckle strength -->
+                    <param name="effort_limit">100.0</param>
                 </state_interface>
             </joint>
@@ -92,5 +105,5 @@
             <joint name="right_inner_knuckle_joint">
                 <state_interface name="position">
-                    <param name="initial_value">${initial_positions['finger_joint']}</param>
+                    <param name="initial_value">${initial_positions['right_inner_knuckle_joint']}</param>
                 </state_interface>
                 <state_interface name="velocity"/>
@@ -102,5 +115,5 @@
             <joint name="left_inner_knuckle_joint">
                 <state_interface name="position">
-                    <param name="initial_value">${initial_positions['finger_joint']}</param>
+                    <param name="initial_value">${initial_positions['left_inner_knuckle_joint']}</param>
                 </state_interface>
                 <state_interface name="velocity"/>
@@ -112,5 +125,5 @@
             <joint name="right_inner_finger_joint">
                 <state_interface name="position">
-                    <param name="initial_value">${initial_positions['finger_joint']}</param>
+                    <param name="initial_value">${initial_positions['right_inner_finger_joint']}</param>
                 </state_interface>
                 <state_interface name="velocity"/>
@@ -122,5 +135,5 @@
             <joint name="left_inner_finger_joint">
                 <state_interface name="position">
-                    <param name="initial_value">${initial_positions['finger_joint']}</param>
+                    <param name="initial_value">${initial_positions['left_inner_finger_joint']}</param>
                 </state_interface>
                 <state_interface name="velocity"/>

Commit message: remove bogus left_outer_knuckle_joint from ros2_control xacro; add obstacles to point_cloud.rviz

File: moveit_config/config/ur.ros2_control.xacro (robot description, xacro)
@@ -81,15 +81,7 @@
                  so Ignition Gazebo initialises every joint individually rather than
                  sharing the finger_joint reference which caused right-side joints to
-                 start at their limit positions). -->
-            <!-- left_outer_knuckle_joint (was missing — added) -->
-            <joint name="left_outer_knuckle_joint">
-                <state_interface name="position">
-                    <param name="initial_value">${initial_positions['left_outer_knuckle_joint']}</param>
-                </state_interface>
-                <state_interface name="velocity"/>
-                <state_interface name="effort">
-                    <param name="effort_limit">100.0</param>
-                </state_interface>
-            </joint>
+                 start at their limit positions).
+                 Note: left_outer_knuckle is driven directly by finger_joint — there
+                 is no separate left_outer_knuckle_joint in the URDF. -->
             <!-- right_outer_knuckle_joint -->
             <joint name="right_outer_knuckle_joint">

Commit message: fix gripper mimic joints: add command_interface with mimic/multiplier params for gz_ros2_control

File: moveit_config/config/ur.ros2_control.xacro (robot description, xacro)
@@ -84,53 +84,62 @@
                  Note: left_outer_knuckle is driven directly by finger_joint — there
                  is no separate left_outer_knuckle_joint in the URDF. -->
-            <!-- right_outer_knuckle_joint -->
+            <!-- Mimic joints: each needs a position command_interface with mimic/multiplier
+                 params so gz_ros2_control emulates the URDF <mimic> constraints in software.
+                 Without this, Ignition Gazebo drops <mimic> tags (they don't exist in SDF)
+                 and only finger_joint moves — all other joints stay frozen. -->
+            <!-- right_outer_knuckle_joint  (multiplier +1) -->
             <joint name="right_outer_knuckle_joint">
+                <command_interface name="position">
+                    <param name="mimic">finger_joint</param>
+                    <param name="multiplier">1</param>
+                </command_interface>
                 <state_interface name="position">
                     <param name="initial_value">${initial_positions['right_outer_knuckle_joint']}</param>
                 </state_interface>
                 <state_interface name="velocity"/>
-                <state_interface name="effort">
-                    <param name="effort_limit">100.0</param>
-                </state_interface>
             </joint>
-            <!-- right_inner_knuckle_joint -->
+            <!-- right_inner_knuckle_joint  (multiplier +1) -->
             <joint name="right_inner_knuckle_joint">
+                <command_interface name="position">
+                    <param name="mimic">finger_joint</param>
+                    <param name="multiplier">1</param>
+                </command_interface>
                 <state_interface name="position">
                     <param name="initial_value">${initial_positions['right_inner_knuckle_joint']}</param>
                 </state_interface>
                 <state_interface name="velocity"/>
-                <state_interface name="effort">
-                    <param name="effort_limit">100.0</param>
-                </state_interface>
             </joint>
-            <!-- left_inner_knuckle_joint -->
+            <!-- left_inner_knuckle_joint  (multiplier +1) -->
             <joint name="left_inner_knuckle_joint">
+                <command_interface name="position">
+                    <param name="mimic">finger_joint</param>
+                    <param name="multiplier">1</param>
+                </command_interface>
                 <state_interface name="position">
                     <param name="initial_value">${initial_positions['left_inner_knuckle_joint']}</param>
                 </state_interface>
                 <state_interface name="velocity"/>
-                <state_interface name="effort">
-                    <param name="effort_limit">100.0</param>
-                </state_interface>
             </joint>
-            <!-- right_inner_finger_joint -->
+            <!-- right_inner_finger_joint  (multiplier -1) -->
             <joint name="right_inner_finger_joint">
+                <command_interface name="position">
+                    <param name="mimic">finger_joint</param>
+                    <param name="multiplier">-1</param>
+                </command_interface>
                 <state_interface name="position">
                     <param name="initial_value">${initial_positions['right_inner_finger_joint']}</param>
                 </state_interface>
                 <state_interface name="velocity"/>
-                <state_interface name="effort">
-                    <param name="effort_limit">100.0</param>
-                </state_interface>
             </joint>
-            <!-- left_inner_finger_joint -->
+            <!-- left_inner_finger_joint  (multiplier -1) -->
             <joint name="left_inner_finger_joint">
+                <command_interface name="position">
+                    <param name="mimic">finger_joint</param>
+                    <param name="multiplier">-1</param>
+                </command_interface>
                 <state_interface name="position">
                     <param name="initial_value">${initial_positions['left_inner_finger_joint']}</param>
                 </state_interface>
                 <state_interface name="velocity"/>
-                <state_interface name="effort">
-                    <param name="effort_limit">100.0</param>
-                </state_interface>
             </joint>
         </ros2_control>

Commit message: revert mimic joints to state_interface only (matches working MTC config)

File: moveit_config/config/ur.ros2_control.xacro (robot description, xacro)
@@ -78,20 +78,18 @@
                 </state_interface>
             </joint>
-            <!-- Mimic joints (no command interfaces, each with explicit initial_value key
-                 so Ignition Gazebo initialises every joint individually rather than
-                 sharing the finger_joint reference which caused right-side joints to
-                 start at their limit positions).
-                 Note: left_outer_knuckle is driven directly by finger_joint — there
-                 is no separate left_outer_knuckle_joint in the URDF. -->
-            <!-- Mimic joints: each needs a position command_interface with mimic/multiplier
-                 params so gz_ros2_control emulates the URDF <mimic> constraints in software.
-                 Without this, Ignition Gazebo drops <mimic> tags (they don't exist in SDF)
-                 and only finger_joint moves — all other joints stay frozen. -->
-            <!-- right_outer_knuckle_joint  (multiplier +1) -->
+            <!-- Mimic joints — state_interface ONLY (no command_interface).
+                 Ignition Gazebo enforces the URDF <mimic> tags natively at the physics
+                 level when the robot is spawned from /robot_description. Adding a
+                 command_interface here fights physics and causes asymmetric finger motion.
+                 Per-joint initial_value keys prevent right-side joints from starting at limits. -->
+            <!-- left_outer_knuckle_joint (was missing — added) -->
+            <joint name="left_outer_knuckle_joint">
+                <state_interface name="position">
+                    <param name="initial_value">${initial_positions['left_outer_knuckle_joint']}</param>
+                </state_interface>
+                <state_interface name="velocity"/>
+            </joint>
+            <!-- right_outer_knuckle_joint -->
             <joint name="right_outer_knuckle_joint">
-                <command_interface name="position">
-                    <param name="mimic">finger_joint</param>
-                    <param name="multiplier">1</param>
-                </command_interface>
                 <state_interface name="position">
                     <param name="initial_value">${initial_positions['right_outer_knuckle_joint']}</param>
@@ -99,10 +97,6 @@
                 <state_interface name="velocity"/>
             </joint>
-            <!-- right_inner_knuckle_joint  (multiplier +1) -->
+            <!-- right_inner_knuckle_joint -->
             <joint name="right_inner_knuckle_joint">
-                <command_interface name="position">
-                    <param name="mimic">finger_joint</param>
-                    <param name="multiplier">1</param>
-                </command_interface>
                 <state_interface name="position">
                     <param name="initial_value">${initial_positions['right_inner_knuckle_joint']}</param>
@@ -110,10 +104,6 @@
                 <state_interface name="velocity"/>
             </joint>
-            <!-- left_inner_knuckle_joint  (multiplier +1) -->
+            <!-- left_inner_knuckle_joint -->
             <joint name="left_inner_knuckle_joint">
-                <command_interface name="position">
-                    <param name="mimic">finger_joint</param>
-                    <param name="multiplier">1</param>
-                </command_interface>
                 <state_interface name="position">
                     <param name="initial_value">${initial_positions['left_inner_knuckle_joint']}</param>
@@ -121,10 +111,6 @@
                 <state_interface name="velocity"/>
             </joint>
-            <!-- right_inner_finger_joint  (multiplier -1) -->
+            <!-- right_inner_finger_joint -->
             <joint name="right_inner_finger_joint">
-                <command_interface name="position">
-                    <param name="mimic">finger_joint</param>
-                    <param name="multiplier">-1</param>
-                </command_interface>
                 <state_interface name="position">
                     <param name="initial_value">${initial_positions['right_inner_finger_joint']}</param>
@@ -132,10 +118,6 @@
                 <state_interface name="velocity"/>
             </joint>
-            <!-- left_inner_finger_joint  (multiplier -1) -->
+            <!-- left_inner_finger_joint -->
             <joint name="left_inner_finger_joint">
-                <command_interface name="position">
-                    <param name="mimic">finger_joint</param>
-                    <param name="multiplier">-1</param>
-                </command_interface>
                 <state_interface name="position">
                     <param name="initial_value">${initial_positions['left_inner_finger_joint']}</param>

Commit message: Fix Robotiq mimic joints in Gazebo Harmonic

File: moveit_config/config/ur.ros2_control.xacro (robot description, xacro)
@@ -78,50 +78,61 @@
                 </state_interface>
             </joint>
-            <!-- Mimic joints — state_interface ONLY (no command_interface).
-                 Ignition Gazebo enforces the URDF <mimic> tags natively at the physics
-                 level when the robot is spawned from /robot_description. Adding a
-                 command_interface here fights physics and causes asymmetric finger motion.
-                 Per-joint initial_value keys prevent right-side joints from starting at limits. -->
-            <!-- left_outer_knuckle_joint (was missing — added) -->
-            <joint name="left_outer_knuckle_joint">
-                <state_interface name="position">
-                    <param name="initial_value">${initial_positions['left_outer_knuckle_joint']}</param>
-                </state_interface>
-                <state_interface name="velocity"/>
-            </joint>
+            <!-- Gazebo Harmonic + DART does not enforce URDF mimic constraints reliably
+                 for this Robotiq model. Mirror the follower joints through
+                 gz_ros2_control instead so the linkage stays coherent at spawn time. -->
             <!-- right_outer_knuckle_joint -->
             <joint name="right_outer_knuckle_joint">
+                <param name="mimic">finger_joint</param>
+                <param name="multiplier">1</param>
+                <command_interface name="position"/>
                 <state_interface name="position">
                     <param name="initial_value">${initial_positions['right_outer_knuckle_joint']}</param>
                 </state_interface>
                 <state_interface name="velocity"/>
+                <state_interface name="effort"/>
             </joint>
             <!-- right_inner_knuckle_joint -->
             <joint name="right_inner_knuckle_joint">
+                <param name="mimic">finger_joint</param>
+                <param name="multiplier">1</param>
+                <command_interface name="position"/>
                 <state_interface name="position">
                     <param name="initial_value">${initial_positions['right_inner_knuckle_joint']}</param>
                 </state_interface>
                 <state_interface name="velocity"/>
+                <state_interface name="effort"/>
             </joint>
             <!-- left_inner_knuckle_joint -->
             <joint name="left_inner_knuckle_joint">
+                <param name="mimic">finger_joint</param>
+                <param name="multiplier">1</param>
+                <command_interface name="position"/>
                 <state_interface name="position">
                     <param name="initial_value">${initial_positions['left_inner_knuckle_joint']}</param>
                 </state_interface>
                 <state_interface name="velocity"/>
+                <state_interface name="effort"/>
             </joint>
             <!-- right_inner_finger_joint -->
             <joint name="right_inner_finger_joint">
+                <param name="mimic">finger_joint</param>
+                <param name="multiplier">-1</param>
+                <command_interface name="position"/>
                 <state_interface name="position">
                     <param name="initial_value">${initial_positions['right_inner_finger_joint']}</param>
                 </state_interface>
                 <state_interface name="velocity"/>
+                <state_interface name="effort"/>
             </joint>
             <!-- left_inner_finger_joint -->
             <joint name="left_inner_finger_joint">
+                <param name="mimic">finger_joint</param>
+                <param name="multiplier">-1</param>
+                <command_interface name="position"/>
                 <state_interface name="position">
                     <param name="initial_value">${initial_positions['left_inner_finger_joint']}</param>
                 </state_interface>
                 <state_interface name="velocity"/>
+                <state_interface name="effort"/>
             </joint>
         </ros2_control>

Commit message: revert mimic joints to state-only in ros2_control xacro

File: moveit_config/config/ur.ros2_control.xacro (robot description, xacro)
@@ -78,61 +78,43 @@
                 </state_interface>
             </joint>
-            <!-- Gazebo Harmonic + DART does not enforce URDF mimic constraints reliably
-                 for this Robotiq model. Mirror the follower joints through
-                 gz_ros2_control instead so the linkage stays coherent at spawn time. -->
-            <!-- right_outer_knuckle_joint -->
+            <!-- Mimic joints — state_interface ONLY (no command_interface).
+                 Gazebo Harmonic enforces URDF <mimic> constraints at the physics level.
+                 Adding command_interface to constrained joints causes GazeboSimSystem
+                 plugin init failure. -->
+            <joint name="left_outer_knuckle_joint">
+                <state_interface name="position">
+                    <param name="initial_value">${initial_positions['left_outer_knuckle_joint']}</param>
+                </state_interface>
+                <state_interface name="velocity"/>
+            </joint>
             <joint name="right_outer_knuckle_joint">
-                <param name="mimic">finger_joint</param>
-                <param name="multiplier">1</param>
-                <command_interface name="position"/>
                 <state_interface name="position">
                     <param name="initial_value">${initial_positions['right_outer_knuckle_joint']}</param>
                 </state_interface>
                 <state_interface name="velocity"/>
-                <state_interface name="effort"/>
             </joint>
-            <!-- right_inner_knuckle_joint -->
             <joint name="right_inner_knuckle_joint">
-                <param name="mimic">finger_joint</param>
-                <param name="multiplier">1</param>
-                <command_interface name="position"/>
                 <state_interface name="position">
                     <param name="initial_value">${initial_positions['right_inner_knuckle_joint']}</param>
                 </state_interface>
                 <state_interface name="velocity"/>
-                <state_interface name="effort"/>
             </joint>
-            <!-- left_inner_knuckle_joint -->
             <joint name="left_inner_knuckle_joint">
-                <param name="mimic">finger_joint</param>
-                <param name="multiplier">1</param>
-                <command_interface name="position"/>
                 <state_interface name="position">
                     <param name="initial_value">${initial_positions['left_inner_knuckle_joint']}</param>
                 </state_interface>
                 <state_interface name="velocity"/>
-                <state_interface name="effort"/>
             </joint>
-            <!-- right_inner_finger_joint -->
             <joint name="right_inner_finger_joint">
-                <param name="mimic">finger_joint</param>
-                <param name="multiplier">-1</param>
-                <command_interface name="position"/>
                 <state_interface name="position">
                     <param name="initial_value">${initial_positions['right_inner_finger_joint']}</param>
                 </state_interface>
                 <state_interface name="velocity"/>
-                <state_interface name="effort"/>
             </joint>
-            <!-- left_inner_finger_joint -->
             <joint name="left_inner_finger_joint">
-                <param name="mimic">finger_joint</param>
-                <param name="multiplier">-1</param>
-                <command_interface name="position"/>
                 <state_interface name="position">
                     <param name="initial_value">${initial_positions['left_inner_finger_joint']}</param>
                 </state_interface>
                 <state_interface name="velocity"/>
-                <state_interface name="effort"/>
             </joint>
         </ros2_control>
