Commit message: add RG2/RG6 and 2F-140 gripper support

File: moveit_config/config/ur.ros2_control.xacro (robot description, xacro)
@@ -1,5 +1,5 @@
 <?xml version="1.0"?>
 <robot xmlns:xacro="http://www.ros.org/wiki/xacro">
-    <xacro:macro name="ur_ros2_control" params="name initial_positions_file">
+    <xacro:macro name="ur_ros2_control" params="name initial_positions_file gripper:=robotiq_2f_85">
         <xacro:property name="initial_positions" value="${xacro.load_yaml(initial_positions_file)['initial_positions']}"/>
         <ros2_control name="${name}" type="system">
@@ -68,54 +68,81 @@
                 </state_interface>
             </joint>
-            <joint name="finger_joint">
-                <command_interface name="position"/>
-                <state_interface name="position">
-                    <param name="initial_value">${initial_positions['finger_joint']}</param>
-                </state_interface>
-                <state_interface name="velocity"/>
-                <state_interface name="effort">
-                    <param name="effort_limit">100.0</param> <!-- Increased effort for finger strength -->
-                </state_interface>
-            </joint>
-            <!-- Mimic joints — state_interface ONLY (no command_interface).
-                 Gazebo Harmonic enforces URDF <mimic> constraints at the physics level.
-                 Adding command_interface to constrained joints causes GazeboSimSystem
-                 plugin init failure. -->
-            <joint name="left_outer_knuckle_joint">
-                <state_interface name="position">
-                    <param name="initial_value">${initial_positions['left_outer_knuckle_joint']}</param>
-                </state_interface>
-                <state_interface name="velocity"/>
-            </joint>
-            <joint name="right_outer_knuckle_joint">
-                <state_interface name="position">
-                    <param name="initial_value">${initial_positions['right_outer_knuckle_joint']}</param>
-                </state_interface>
-                <state_interface name="velocity"/>
-            </joint>
-            <joint name="right_inner_knuckle_joint">
-                <state_interface name="position">
-                    <param name="initial_value">${initial_positions['right_inner_knuckle_joint']}</param>
-                </state_interface>
-                <state_interface name="velocity"/>
-            </joint>
-            <joint name="left_inner_knuckle_joint">
-                <state_interface name="position">
-                    <param name="initial_value">${initial_positions['left_inner_knuckle_joint']}</param>
-                </state_interface>
-                <state_interface name="velocity"/>
-            </joint>
-            <joint name="right_inner_finger_joint">
-                <state_interface name="position">
-                    <param name="initial_value">${initial_positions['right_inner_finger_joint']}</param>
-                </state_interface>
-                <state_interface name="velocity"/>
-            </joint>
-            <joint name="left_inner_finger_joint">
-                <state_interface name="position">
-                    <param name="initial_value">${initial_positions['left_inner_finger_joint']}</param>
-                </state_interface>
-                <state_interface name="velocity"/>
-            </joint>
+            <xacro:if value="${gripper == 'robotiq_2f_85' or gripper == 'robotiq_2f_140'}">
+                <joint name="finger_joint">
+                    <command_interface name="position"/>
+                    <state_interface name="position">
+                        <param name="initial_value">${initial_positions['finger_joint']}</param>
+                    </state_interface>
+                    <state_interface name="velocity"/>
+                    <state_interface name="effort">
+                        <param name="effort_limit">100.0</param>
+                    </state_interface>
+                </joint>
+                <!-- Mimic joints — state_interface ONLY (no command_interface).
+                     Gazebo Harmonic enforces URDF <mimic> constraints at the physics level.
+                     Adding command_interface to constrained joints causes GazeboSimSystem
+                     plugin init failure. -->
+                <joint name="left_outer_knuckle_joint">
+                    <state_interface name="position">
+                        <param name="initial_value">${initial_positions['left_outer_knuckle_joint']}</param>
+                    </state_interface>
+                    <state_interface name="velocity"/>
+                </joint>
+                <joint name="right_outer_knuckle_joint">
+                    <state_interface name="position">
+                        <param name="initial_value">${initial_positions['right_outer_knuckle_joint']}</param>
+                    </state_interface>
+                    <state_interface name="velocity"/>
+                </joint>
+                <joint name="right_inner_knuckle_joint">
+                    <state_interface name="position">
+                        <param name="initial_value">${initial_positions['right_inner_knuckle_joint']}</param>
+                    </state_interface>
+                    <state_interface name="velocity"/>
+                </joint>
+                <joint name="left_inner_knuckle_joint">
+                    <state_interface name="position">
+                        <param name="initial_value">${initial_positions['left_inner_knuckle_joint']}</param>
+                    </state_interface>
+                    <state_interface name="velocity"/>
+                </joint>
+                <joint name="right_inner_finger_joint">
+                    <state_interface name="position">
+                        <param name="initial_value">${initial_positions['right_inner_finger_joint']}</param>
+                    </state_interface>
+                    <state_interface name="velocity"/>
+                </joint>
+                <joint name="left_inner_finger_joint">
+                    <state_interface name="position">
+                        <param name="initial_value">${initial_positions['left_inner_finger_joint']}</param>
+                    </state_interface>
+                    <state_interface name="velocity"/>
+                </joint>
+            </xacro:if>
+            <xacro:if value="${gripper == 'onrobot_rg2' or gripper == 'onrobot_rg6'}">
+                <joint name="gripper_joint">
+                    <command_interface name="position"/>
+                    <state_interface name="position">
+                        <param name="initial_value">${initial_positions['gripper_joint']}</param>
+                    </state_interface>
+                    <state_interface name="velocity"/>
+                    <state_interface name="effort"/>
+                </joint>
+                <joint name="gripper_finger_1_truss_arm_joint">
+                    <state_interface name="position"/>
+                </joint>
+                <joint name="gripper_finger_1_finger_tip_joint">
+                    <state_interface name="position"/>
+                </joint>
+                <joint name="gripper_mirror_joint">
+                    <state_interface name="position"/>
+                </joint>
+                <joint name="gripper_finger_2_truss_arm_joint">
+                    <state_interface name="position"/>
+                </joint>
+                <joint name="gripper_finger_2_finger_tip_joint">
+                    <state_interface name="position"/>
+                </joint>
+            </xacro:if>
         </ros2_control>
     </xacro:macro>

File: moveit_config/config/ur.urdf.xacro (robot description, xacro)
@@ -19,4 +19,9 @@
     <xacro:include filename="$(find moveit_config)/config/ur.ros2_control.xacro" />
     <xacro:include filename="$(find ur_description)/urdf/gazebo_sim_ros2_control.urdf.xacro" />
+    <xacro:property name="selected_gripper" value="$(arg gripper)"/>
+    <xacro:property name="controllers_file" value="$(find moveit_config)/config/ros2_controllers.yaml"/>
+    <xacro:if value="${selected_gripper == 'onrobot_rg2' or selected_gripper == 'onrobot_rg6'}">
+      <xacro:property name="controllers_file" value="$(find moveit_config)/config/ros2_controllers_onrobot.yaml"/>
+    </xacro:if>
     <link name="world" />
     <xacro:ur_robot
@@ -38,8 +43,12 @@
       <disableFixedJointLumping>true</disableFixedJointLumping>
     </gazebo>
-    <xacro:ur_ros2_control name="ur" initial_positions_file="$(find moveit_config)/config/initial_positions.yaml"/>
+    <xacro:ur_ros2_control
+      name="ur"
+      initial_positions_file="$(find moveit_config)/config/initial_positions.yaml"
+      gripper="$(arg gripper)"/>
     <xacro:load_gazebo_sim_ros2_control_plugin
       robot_name="$(arg robot_name)"
-      use_gazebo="$(arg use_gazebo)"/>
+      use_gazebo="$(arg use_gazebo)"
+      controllers_file="${controllers_file}"/>
     <xacro:include filename="$(find ur_description)/urdf/intel_rgbd_cam_d435.urdf.xacro"/>
 </robot>

File: onrobot_description/urdf/onrobot_rg.urdf.xacro (robot description, xacro)
@@ -9,5 +9,5 @@
   <!-- onrobot gripper -->
   <xacro:macro name="onrobot_rg" params="parent *origin prefix:=''
-    model:='rg2_v1' safety_shield:=False bracket:='single_bracket' mount_angle:=0.0 standalone:=false real_hardware:=false">
+    model:='rg2_v1' safety_shield:=False bracket:='single_bracket' mount_angle:=0.0 standalone:=false real_hardware:=false include_ros2_control:=true">
     <xacro:property name="gripper_name" value="${prefix}gripper"/>
     <!-- load config from file -->
@@ -219,4 +219,5 @@
     <xacro:finger name="${gripper_name}_finger_1" is_master="true"/>
     <xacro:finger name="${gripper_name}_finger_2" is_master="false"/>
+    <xacro:if value="${include_ros2_control}">
     <ros2_control name="${gripper_name}" type="system" is_async="true">
           <xacro:unless value="${real_hardware}">
@@ -269,4 +270,5 @@
           </xacro:if>
     </ros2_control>
+    </xacro:if>
     <!-- si standalone alors mettre le plugin de ros2_control -->
     <xacro:unless value="${real_hardware}">

File: ur_description/urdf/ur_macro.xacro (robot description, xacro)
@@ -355,5 +355,5 @@
   <!-- OnRobot RG2 -->
   <xacro:if value="${gripper == 'onrobot_rg2'}">
-    <xacro:onrobot_rg prefix="" model="rg2_v1" parent="${tf_prefix}tool0" standalone="false">
+    <xacro:onrobot_rg prefix="" model="rg2_v1" parent="${tf_prefix}tool0" standalone="false" include_ros2_control="false">
       <origin xyz="0 0 0.01" rpy="0 0 ${pi/2}"/>
     </xacro:onrobot_rg>
@@ -361,5 +361,5 @@
   <!-- OnRobot RG6 -->
   <xacro:if value="${gripper == 'onrobot_rg6'}">
-    <xacro:onrobot_rg prefix="" model="rg6_v1" parent="${tf_prefix}tool0" standalone="false">
+    <xacro:onrobot_rg prefix="" model="rg6_v1" parent="${tf_prefix}tool0" standalone="false" include_ros2_control="false">
       <origin xyz="0 0 0.01" rpy="0 0 ${pi/2}"/>
     </xacro:onrobot_rg>

Commit message: drop ghost knuckle joint

File: moveit_config/config/ur.ros2_control.xacro (robot description, xacro)
@@ -80,13 +80,6 @@
                 </joint>
                 <!-- Mimic joints — state_interface ONLY (no command_interface).
-                     Gazebo Harmonic enforces URDF <mimic> constraints at the physics level.
                      Adding command_interface to constrained joints causes GazeboSimSystem
                      plugin init failure. -->
-                <joint name="left_outer_knuckle_joint">
-                    <state_interface name="position">
-                        <param name="initial_value">${initial_positions['left_outer_knuckle_joint']}</param>
-                    </state_interface>
-                    <state_interface name="velocity"/>
-                </joint>
                 <joint name="right_outer_knuckle_joint">
                     <state_interface name="position">
