Commit message: add dual arm moveit support and fixes

File: moveit_config/config/ur.ros2_control.xacro (robot description, xacro)
@@ -1,5 +1,5 @@
 <?xml version="1.0"?>
 <robot xmlns:xacro="http://www.ros.org/wiki/xacro">
-    <xacro:macro name="ur_ros2_control" params="name initial_positions_file gripper:=robotiq_2f_85">
+    <xacro:macro name="ur_ros2_control" params="name initial_positions_file gripper:=robotiq_2f_85 prefix:=''">
         <xacro:property name="initial_positions" value="${xacro.load_yaml(initial_positions_file)['initial_positions']}"/>
         <ros2_control name="${name}" type="system">
@@ -8,5 +8,5 @@
                 <plugin>gz_ros2_control/GazeboSimSystem</plugin>
             </hardware>
-            <joint name="shoulder_pan_joint">
+            <joint name="${prefix}shoulder_pan_joint">
                 <command_interface name="position"/>
                 <command_interface name="effort">
@@ -22,5 +22,5 @@
                 </state_interface>
             </joint>
-            <joint name="shoulder_lift_joint">
+            <joint name="${prefix}shoulder_lift_joint">
                 <command_interface name="position"/>
                 <command_interface name="effort">
@@ -36,5 +36,5 @@
                 </state_interface>
             </joint>
-            <joint name="elbow_joint">
+            <joint name="${prefix}elbow_joint">
                 <command_interface name="position"/>
                 <command_interface name="effort">
@@ -50,5 +50,5 @@
                 </state_interface>
             </joint>
-            <joint name="wrist_1_joint">
+            <joint name="${prefix}wrist_1_joint">
                 <command_interface name="position"/>
                 <command_interface name="effort">
@@ -64,5 +64,5 @@
                 </state_interface>
             </joint>
-            <joint name="wrist_2_joint">
+            <joint name="${prefix}wrist_2_joint">
                 <command_interface name="position"/>
                 <command_interface name="effort">
@@ -78,5 +78,5 @@
                 </state_interface>
             </joint>
-            <joint name="wrist_3_joint">
+            <joint name="${prefix}wrist_3_joint">
                 <command_interface name="position"/>
                 <command_interface name="effort">
@@ -93,5 +93,5 @@
             </joint>
             <xacro:if value="${gripper == 'robotiq_2f_85' or gripper == 'robotiq_2f_140'}">
-                <joint name="finger_joint">
+                <joint name="${prefix}finger_joint">
                     <command_interface name="position"/>
                     <state_interface name="position">
@@ -106,5 +106,5 @@
                      Adding command_interface to constrained joints causes GazeboSimSystem
                      plugin init failure. -->
-                <joint name="right_outer_knuckle_joint">
+                <joint name="${prefix}right_outer_knuckle_joint">
                     <state_interface name="position">
                         <param name="initial_value">${initial_positions['right_outer_knuckle_joint']}</param>
@@ -112,5 +112,5 @@
                     <state_interface name="velocity"/>
                 </joint>
-                <joint name="right_inner_knuckle_joint">
+                <joint name="${prefix}right_inner_knuckle_joint">
                     <state_interface name="position">
                         <param name="initial_value">${initial_positions['right_inner_knuckle_joint']}</param>
@@ -118,5 +118,5 @@
                     <state_interface name="velocity"/>
                 </joint>
-                <joint name="left_inner_knuckle_joint">
+                <joint name="${prefix}left_inner_knuckle_joint">
                     <state_interface name="position">
                         <param name="initial_value">${initial_positions['left_inner_knuckle_joint']}</param>
@@ -124,5 +124,5 @@
                     <state_interface name="velocity"/>
                 </joint>
-                <joint name="right_inner_finger_joint">
+                <joint name="${prefix}right_inner_finger_joint">
                     <state_interface name="position">
                         <param name="initial_value">${initial_positions['right_inner_finger_joint']}</param>
@@ -130,5 +130,5 @@
                     <state_interface name="velocity"/>
                 </joint>
-                <joint name="left_inner_finger_joint">
+                <joint name="${prefix}left_inner_finger_joint">
                     <state_interface name="position">
                         <param name="initial_value">${initial_positions['left_inner_finger_joint']}</param>
@@ -138,5 +138,5 @@
             </xacro:if>
             <xacro:if value="${gripper == 'onrobot_rg2' or gripper == 'onrobot_rg6'}">
-                <joint name="gripper_joint">
+                <joint name="${prefix}gripper_joint">
                     <command_interface name="position"/>
                     <state_interface name="position">
@@ -146,17 +146,17 @@
                     <state_interface name="effort"/>
                 </joint>
-                <joint name="gripper_finger_1_truss_arm_joint">
+                <joint name="${prefix}gripper_finger_1_truss_arm_joint">
                     <state_interface name="position"/>
                 </joint>
-                <joint name="gripper_finger_1_finger_tip_joint">
+                <joint name="${prefix}gripper_finger_1_finger_tip_joint">
                     <state_interface name="position"/>
                 </joint>
-                <joint name="gripper_mirror_joint">
+                <joint name="${prefix}gripper_mirror_joint">
                     <state_interface name="position"/>
                 </joint>
-                <joint name="gripper_finger_2_truss_arm_joint">
+                <joint name="${prefix}gripper_finger_2_truss_arm_joint">
                     <state_interface name="position"/>
                 </joint>
-                <joint name="gripper_finger_2_finger_tip_joint">
+                <joint name="${prefix}gripper_finger_2_finger_tip_joint">
                     <state_interface name="position"/>
                 </joint>

File: ur_description/urdf/ur_macro.xacro (robot description, xacro)
@@ -339,5 +339,5 @@
   <!-- Robotiq 2F-85 -->
   <xacro:if value="${gripper == 'robotiq_2f_85'}">
-    <xacro:robotiq_arg2f_85 prefix=""/>
+    <xacro:robotiq_arg2f_85 prefix="${tf_prefix}"/>
     <joint name="${tf_prefix}gripper_joint" type="fixed">
       <parent link="${tf_prefix}tool0"/>
@@ -349,5 +349,5 @@
   <!-- Robotiq 2F-140 -->
   <xacro:if value="${gripper == 'robotiq_2f_140'}">
-    <xacro:robotiq_gripper name="robotiq_140" prefix="" parent="${tf_prefix}tool0" include_ros2_control="false">
+    <xacro:robotiq_gripper name="${tf_prefix}robotiq_140" prefix="${tf_prefix}" parent="${tf_prefix}tool0" include_ros2_control="false">
       <origin xyz="0 0 0.01" rpy="0 0 0"/>
     </xacro:robotiq_gripper>
@@ -355,5 +355,5 @@
   <!-- OnRobot RG2 -->
   <xacro:if value="${gripper == 'onrobot_rg2'}">
-    <xacro:onrobot_rg prefix="" model="rg2_v1" parent="${tf_prefix}tool0" standalone="false" include_ros2_control="false">
+    <xacro:onrobot_rg prefix="${tf_prefix}" model="rg2_v1" parent="${tf_prefix}tool0" standalone="false" include_ros2_control="false">
       <origin xyz="0 0 0.01" rpy="0 0 ${pi/2}"/>
     </xacro:onrobot_rg>
@@ -361,5 +361,5 @@
   <!-- OnRobot RG6 -->
   <xacro:if value="${gripper == 'onrobot_rg6'}">
-    <xacro:onrobot_rg prefix="" model="rg6_v1" parent="${tf_prefix}tool0" standalone="false" include_ros2_control="false">
+    <xacro:onrobot_rg prefix="${tf_prefix}" model="rg6_v1" parent="${tf_prefix}tool0" standalone="false" include_ros2_control="false">
       <origin xyz="0 0 0.01" rpy="0 0 ${pi/2}"/>
     </xacro:onrobot_rg>
