Commit message: dual-arm per-arm pipelines

File: moveit_config/config/dual_ur.srdf.xacro (robot description, xacro)
@@ -2,15 +2,15 @@
 <!--
 Dual-arm semantic description for dual_ur.urdf.xacro. Mirrors ur.srdf.xacro's
-robotiq_2f_85/2f_140 branch, but wrapped in a macro parameterized on `prefix`
-("left_"/"right_") and instantiated once per arm, so each arm gets its own
-{prefix}arm / {prefix}gripper / {prefix}arm_with_gripper planning groups
-instead of colliding on "arm"/"gripper". No camera links: dual_ur.urdf.xacro
-doesn't include cameras yet (see its header comment).
-Only supports the robotiq_2f_85/2f_140 grippers for now, matching the two
-grippers dual_ur.urdf.xacro's onrobot branch was never written for (phase 1
-only tested robotiq grippers on the dual rig).
+gripper branches (robotiq_2f_85/2f_140 and onrobot_rg2/rg6), but wrapped in a
+macro parameterized on `prefix` ("left_"/"right_") and instantiated once per
+arm, so each arm gets its own {prefix}arm / {prefix}gripper /
+{prefix}arm_with_gripper planning groups instead of colliding on "arm"/"gripper".
+Camera disable_collisions entries only apply when use_dual_cameras:=true
+(dual_ur.urdf.xacro's opt-in camera instantiation), default false, matching
+dual_ur.urdf.xacro's default, so nothing changes for existing (no-camera) use.
 -->
 <robot xmlns:xacro="http://www.ros.org/wiki/xacro" name="dual_ur">
     <xacro:arg name="gripper" default="robotiq_2f_85"/>
+    <xacro:arg name="use_dual_cameras" default="false"/>
     <xacro:property name="selected_gripper" value="$(arg gripper)"/>
     <xacro:property name="gripper_base_link" value="${'robotiq_140_base_link' if selected_gripper == 'robotiq_2f_140' else 'robotiq_arg2f_base_link'}"/>
@@ -22,18 +22,7 @@
     <!--SUBGROUPS: Groups can also be formed by referencing to already defined group names-->
     <group name="${prefix}arm">
-        <!-- <joint name="${prefix}base_joint"/>
-        <joint name="base_link-base_fixed_joint"/>
-        <joint name="base_link-base_link_inertia"/>
-        <joint name="${prefix}shoulder_pan_joint"/>
-        <joint name="${prefix}shoulder_lift_joint"/>
-        <joint name="${prefix}elbow_joint"/>
-        <joint name="${prefix}wrist_1_joint"/>
-        <joint name="${prefix}wrist_2_joint"/>
-        <joint name="${prefix}wrist_3_joint"/>
-        <joint name="wrist_3-flange"/>
-        <joint name="flange-tool0"/>
-        <joint name="${prefix}gripper_joint"/> -->
         <chain base_link="world" tip_link="${prefix}tool0"/>
     </group>
+    <xacro:if value="${selected_gripper == 'robotiq_2f_85' or selected_gripper == 'robotiq_2f_140'}">
     <group name="${prefix}gripper">
         <joint name="${prefix}finger_joint"/>
@@ -226,4 +215,97 @@
     <disable_collisions link1="${prefix}shoulder_link" link2="${prefix}right_outer_knuckle" reason="Never"/>
     <disable_collisions link1="${prefix}shoulder_link" link2="${prefix}${gripper_base_link}" reason="Never"/>
+    </xacro:if>
+    <xacro:unless value="${selected_gripper == 'robotiq_2f_85' or selected_gripper == 'robotiq_2f_140'}">
+    <group name="${prefix}gripper">
+        <joint name="${prefix}gripper_joint"/>
+    </group>
+    <group name="${prefix}arm_with_gripper">
+        <group name="${prefix}gripper"/>
+        <group name="${prefix}arm"/>
+    </group>
+    <group_state name="home" group="${prefix}arm">
+        <joint name="${prefix}elbow_joint" value="0"/>
+        <joint name="${prefix}shoulder_lift_joint" value="-1.6663"/>
+        <joint name="${prefix}shoulder_pan_joint" value="0"/>
+        <joint name="${prefix}wrist_1_joint" value="0"/>
+        <joint name="${prefix}wrist_2_joint" value="0"/>
+        <joint name="${prefix}wrist_3_joint" value="0"/>
+    </group_state>
+    <group_state name="ready" group="${prefix}arm">
+        <joint name="${prefix}elbow_joint" value="0"/>
+        <joint name="${prefix}shoulder_lift_joint" value="-1.6663"/>
+        <joint name="${prefix}shoulder_pan_joint" value="0"/>
+        <joint name="${prefix}wrist_1_joint" value="0"/>
+        <joint name="${prefix}wrist_2_joint" value="0"/>
+        <joint name="${prefix}wrist_3_joint" value="1.0"/>
+    </group_state>
+    <!-- FK-screened joint-space via: tool0 ≈ (0.17, 0.00, 0.67), clear of
+         the pick-table AABB between base and object. -->
+    <group_state name="transit_clear" group="${prefix}arm">
+        <!-- Rescreened: tool0≈(0.18,0.08,0.64), pan≈0 keeps gripper clear of torso. -->
+        <joint name="${prefix}shoulder_pan_joint" value="-0.09"/>
+        <joint name="${prefix}shoulder_lift_joint" value="-0.72"/>
+        <joint name="${prefix}elbow_joint" value="-0.84"/>
+        <joint name="${prefix}wrist_1_joint" value="-0.98"/>
+        <joint name="${prefix}wrist_2_joint" value="1.79"/>
+        <joint name="${prefix}wrist_3_joint" value="-0.04"/>
+    </group_state>
+    <group_state name="open" group="${prefix}gripper">
+        <joint name="${prefix}gripper_joint" value="0.0"/>
+    </group_state>
+    <group_state name="half_closed" group="${prefix}gripper">
+        <joint name="${prefix}gripper_joint" value="0.65"/>
+    </group_state>
+    <group_state name="closed" group="${prefix}gripper">
+        <joint name="${prefix}gripper_joint" value="1.3"/>
+    </group_state>
+    <end_effector name="${prefix}gripper" parent_link="${prefix}tool0" group="${prefix}gripper" parent_group="${prefix}arm"/>
+    <disable_collisions link1="${prefix}base_link_inertia" link2="${prefix}shoulder_link" reason="Adjacent"/>
+    <disable_collisions link1="${prefix}forearm_link" link2="${prefix}upper_arm_link" reason="Adjacent"/>
+    <disable_collisions link1="${prefix}forearm_link" link2="${prefix}wrist_1_link" reason="Adjacent"/>
+    <disable_collisions link1="${prefix}forearm_link" link2="${prefix}wrist_2_link" reason="Never"/>
+    <disable_collisions link1="${prefix}shoulder_link" link2="${prefix}upper_arm_link" reason="Adjacent"/>
+    <disable_collisions link1="${prefix}shoulder_link" link2="${prefix}wrist_1_link" reason="Never"/>
+    <disable_collisions link1="${prefix}shoulder_link" link2="${prefix}wrist_2_link" reason="Never"/>
+    <disable_collisions link1="${prefix}wrist_1_link" link2="${prefix}wrist_2_link" reason="Adjacent"/>
+    <disable_collisions link1="${prefix}wrist_1_link" link2="${prefix}wrist_3_link" reason="Never"/>
+    <disable_collisions link1="${prefix}wrist_2_link" link2="${prefix}wrist_3_link" reason="Adjacent"/>
+    <disable_collisions link1="${prefix}tool0" link2="${prefix}gripper_bracket" reason="Adjacent"/>
+    <disable_collisions link1="${prefix}gripper_bracket" link2="${prefix}gripper_body" reason="Adjacent"/>
+    <disable_collisions link1="${prefix}gripper_body" link2="${prefix}gripper_finger_1_origin" reason="Adjacent"/>
+    <disable_collisions link1="${prefix}gripper_body" link2="${prefix}gripper_finger_2_origin" reason="Adjacent"/>
+    <disable_collisions link1="${prefix}gripper_finger_1_origin" link2="${prefix}gripper_finger_1_moment_arm" reason="Adjacent"/>
+    <disable_collisions link1="${prefix}gripper_finger_1_origin" link2="${prefix}gripper_finger_1_truss_arm" reason="Adjacent"/>
+    <disable_collisions link1="${prefix}gripper_finger_2_origin" link2="${prefix}gripper_finger_2_moment_arm" reason="Adjacent"/>
+    <disable_collisions link1="${prefix}gripper_finger_2_origin" link2="${prefix}gripper_finger_2_truss_arm" reason="Adjacent"/>
+    <disable_collisions link1="${prefix}gripper_finger_1_truss_arm" link2="${prefix}gripper_finger_1_finger_tip" reason="Adjacent"/>
+    <disable_collisions link1="${prefix}gripper_finger_2_truss_arm" link2="${prefix}gripper_finger_2_finger_tip" reason="Adjacent"/>
+    <disable_collisions link1="${prefix}gripper_finger_1_finger_tip" link2="${prefix}gripper_finger_1_flex_finger" reason="Adjacent"/>
+    <disable_collisions link1="${prefix}gripper_finger_2_finger_tip" link2="${prefix}gripper_finger_2_flex_finger" reason="Adjacent"/>
+    <disable_collisions link1="${prefix}gripper_body" link2="${prefix}wrist_3_link" reason="Never"/>
+    <disable_collisions link1="${prefix}gripper_bracket" link2="${prefix}wrist_3_link" reason="Adjacent"/>
+    </xacro:unless>
+    <!-- Camera mount disable_collisions, only relevant when dual_ur.urdf.xacro
+         is built with use_dual_cameras:=true (default false, no-op otherwise). -->
+    <xacro:if value="$(arg use_dual_cameras)">
+    <disable_collisions link1="${prefix}base_link_inertia" link2="${prefix}camera_head_link" reason="Never"/>
+    <disable_collisions link1="${prefix}base_link_inertia" link2="${prefix}torso_link" reason="Adjacent"/>
+    <disable_collisions link1="${prefix}camera_head_link" link2="${prefix}shoulder_link" reason="Never"/>
+    <disable_collisions link1="${prefix}camera_head_link" link2="${prefix}torso_link" reason="Adjacent"/>
+    <disable_collisions link1="${prefix}camera_head_link" link2="${prefix}upper_arm_link" reason="Never"/>
+    </xacro:if>
+    <!-- TODO: placeholder, needs offline IK once a physical handover pose is
+         chosen (see project plan). Values below are NOT a real
+         reachable/collision-checked target, do not command this state
+         until replaced with real numbers derived from a chosen handover
+         Cartesian pose. -->
+    <group_state name="handover" group="${prefix}arm">
+        <joint name="${prefix}elbow_joint" value="0"/>
+        <joint name="${prefix}shoulder_lift_joint" value="0"/>
+        <joint name="${prefix}shoulder_pan_joint" value="0"/>
+        <joint name="${prefix}wrist_1_joint" value="0"/>
+        <joint name="${prefix}wrist_2_joint" value="0"/>
+        <joint name="${prefix}wrist_3_joint" value="0"/>
+    </group_state>
     </xacro:macro>
     <xacro:dual_ur_arm_semantics prefix="left_"/>
@@ -236,3 +318,20 @@
         <group name="right_arm"/>
     </group>
+    <!-- Both arms simultaneously at their existing per-arm "home" joint
+         values, a genuine both_arms-group target, no new numbers guessed,
+         just the per-arm home values above concatenated. -->
+    <group_state name="both_home" group="both_arms">
+        <joint name="left_elbow_joint" value="0"/>
+        <joint name="left_shoulder_lift_joint" value="-1.6663"/>
+        <joint name="left_shoulder_pan_joint" value="0"/>
+        <joint name="left_wrist_1_joint" value="0"/>
+        <joint name="left_wrist_2_joint" value="0"/>
+        <joint name="left_wrist_3_joint" value="0"/>
+        <joint name="right_elbow_joint" value="0"/>
+        <joint name="right_shoulder_lift_joint" value="-1.6663"/>
+        <joint name="right_shoulder_pan_joint" value="0"/>
+        <joint name="right_wrist_1_joint" value="0"/>
+        <joint name="right_wrist_2_joint" value="0"/>
+        <joint name="right_wrist_3_joint" value="0"/>
+    </group_state>
 </robot>

File: moveit_config/config/dual_ur.urdf.xacro (robot description, xacro)
@@ -3,8 +3,7 @@
 Dual-arm variant of ur.urdf.xacro — two independent UR3 arms ("left_"/"right_"
 tf_prefix) on one world link, sharing a single ros2_control plugin/controller_manager.
-Phase 1: independent arm motion only, no MoveIt/SRDF wiring yet (see dual_ur.gazebo.launch.py).
-No cameras yet — ur_description's camera xacros use a single global `$(arg prefix)`,
-not a macro param, so they can only be included once per file; adding dual cameras
-needs those xacros converted to proper macros first.
+Phase 2: independent arm motion, per-arm MoveIt groups (see dual_ur.srdf.xacro),
+onrobot_rg2/rg6 gripper support, and opt-in dual cameras (use_dual_cameras:=true)
+now supported — see dual_ur.gazebo.launch.py.
 -->
 <robot xmlns:xacro="http://www.ros.org/wiki/xacro" name="dual_ur">
@@ -25,9 +24,16 @@
     <xacro:arg name="left_y" default="0.45"/>
     <xacro:arg name="right_y" default="-0.45"/>
+    <!-- Opt-in per-arm D435 head camera (default off, matches dual_ur.srdf.xacro's
+         same-named arg for its camera-mount disable_collisions entries). -->
+    <xacro:arg name="use_dual_cameras" default="false"/>
     <xacro:include filename="$(find ur_description)/urdf/ur_macro.xacro" />
     <xacro:include filename="$(find moveit_config)/config/ur.ros2_control.xacro" />
     <xacro:include filename="$(find ur_description)/urdf/gazebo_sim_ros2_control.urdf.xacro" />
+    <xacro:include filename="$(find ur_description)/urdf/intel_rgbd_cam_d435.urdf.xacro" />
     <xacro:property name="selected_gripper" value="$(arg gripper)"/>
     <xacro:property name="controllers_file" value="$(find moveit_config)/config/dual_ros2_controllers.yaml"/>
+    <xacro:if value="${selected_gripper == 'onrobot_rg2' or selected_gripper == 'onrobot_rg6'}">
+      <xacro:property name="controllers_file" value="$(find moveit_config)/config/dual_ros2_controllers_onrobot.yaml"/>
+    </xacro:if>
     <link name="world" />
     <!-- bullet-featherstone (default physics engine) only supports ONE
@@ -76,4 +82,8 @@
       <disableFixedJointLumping>true</disableFixedJointLumping>
     </gazebo>
+    <xacro:if value="$(arg use_dual_cameras)">
+      <xacro:intel_rgbd_cam_d435 prefix="left_" parent_link="left_base_link"/>
+      <xacro:intel_rgbd_cam_d435 prefix="right_" parent_link="right_base_link"/>
+    </xacro:if>
     <xacro:ur_ros2_control
       name="left_ur"

File: moveit_config/config/ur.urdf.xacro (robot description, xacro)
@@ -53,4 +53,5 @@
       controllers_file="${controllers_file}"/>
     <xacro:include filename="$(find ur_description)/urdf/intel_rgbd_cam_d435.urdf.xacro"/>
+    <xacro:intel_rgbd_cam_d435 prefix="$(arg tf_prefix)" parent_link="$(arg tf_prefix)base_link"/>
     <xacro:include filename="$(find ur_description)/urdf/intel_rgbd_cam_d435_wrist.urdf.xacro"/>
 </robot>

File: ur_description/urdf/intel_rgbd_cam_d435.urdf.xacro (robot description, xacro)
@@ -3,5 +3,8 @@
   <xacro:arg name="use_camera" default="true"/>
   <xacro:arg name="use_gazebo" default="true"/>
-  <xacro:arg name="prefix" default=""/>
+  <!-- prefix: tf_prefix of the arm this camera mounts to ("left_"/"right_"/"").
+       parent_link: the arm link the camera's torso mount attaches to
+       (defaults to "base_link", matching single-arm's unprefixed usage). -->
+  <xacro:macro name="intel_rgbd_cam_d435" params="prefix:='' parent_link:='base_link'">
   <xacro:if value="${'true' == '$(arg use_camera)' and 'true' == '$(arg use_gazebo)'}">
     <xacro:property name="M_PI" value="3.1415926535897931" />
@@ -13,5 +16,5 @@
     <xacro:property name="d435_cam_depth_to_color_offset" value="0.015"/>
     <xacro:property name="camera_tilt_angle_deg" value="55"/>
-  <link name="torso_link">
+  <link name="${prefix}torso_link">
   <inertial>
     <origin xyz="0 0 0.60" />
@@ -50,15 +53,15 @@
   </collision>
 </link>
-    <joint name="$(arg prefix)base_link_to_torso_link" type="fixed">
-      <parent link="$(arg prefix)base_link"/>
-      <child link="torso_link"/>
+    <joint name="${prefix}base_link_to_torso_link" type="fixed">
+      <parent link="${parent_link}"/>
+      <child link="${prefix}torso_link"/>
       <origin xyz="0.22 -0.30 0" rpy="0 0 0"/>
     </joint>
-    <joint name="camera_head_joint" type="fixed">
-      <parent link="torso_link"/>
-      <child link="camera_head_link" />
+    <joint name="${prefix}camera_head_joint" type="fixed">
+      <parent link="${prefix}torso_link"/>
+      <child link="${prefix}camera_head_link" />
       <origin xyz="0 0.01 0.70" rpy="0.0 ${camera_tilt_angle_deg * M_PI / 180} ${M_PI/2}"/>
     </joint>
-    <link name="camera_head_link">
+    <link name="${prefix}camera_head_link">
       <visual>
         <origin xyz="0 0 0" rpy="${M_PI/2} 0.0 ${M_PI/2}"/>
@@ -82,54 +85,54 @@
       </inertial>
     </link>
-    <joint name="camera_head_depth_joint" type="fixed">
+    <joint name="${prefix}camera_head_depth_joint" type="fixed">
       <origin xyz="0 0 0" rpy="0 0 0"/>
-      <parent link="camera_head_link"/>
-      <child link="camera_head_depth_frame" />
+      <parent link="${prefix}camera_head_link"/>
+      <child link="${prefix}camera_head_depth_frame" />
     </joint>
-    <link name="camera_head_depth_frame"/>
-    <joint name="camera_head_depth_optical_joint" type="fixed">
+    <link name="${prefix}camera_head_depth_frame"/>
+    <joint name="${prefix}camera_head_depth_optical_joint" type="fixed">
       <origin xyz="0 0 0" rpy="${-M_PI/2} 0 ${-M_PI/2}" />
-      <parent link="camera_head_depth_frame" />
-      <child link="camera_head_depth_optical_frame" />
+      <parent link="${prefix}camera_head_depth_frame" />
+      <child link="${prefix}camera_head_depth_optical_frame" />
     </joint>
-    <link name="camera_head_depth_optical_frame"/>
-    <joint name="camera_head_infra1_joint" type="fixed">
+    <link name="${prefix}camera_head_depth_optical_frame"/>
+    <joint name="${prefix}camera_head_infra1_joint" type="fixed">
       <origin xyz="0 ${d435_cam_depth_to_infra1_offset} 0" rpy="0 0 0" />
-      <parent link="camera_head_link" />
-      <child link="camera_head_infra1_frame" />
+      <parent link="${prefix}camera_head_link" />
+      <child link="${prefix}camera_head_infra1_frame" />
     </joint>
-    <link name="camera_head_infra1_frame"/>
-    <joint name="camera_head_infra1_optical_joint" type="fixed">
+    <link name="${prefix}camera_head_infra1_frame"/>
+    <joint name="${prefix}camera_head_infra1_optical_joint" type="fixed">
       <origin xyz="0 0 0" rpy="${-M_PI/2} 0 ${-M_PI/2}" />
-      <parent link="camera_head_infra1_frame" />
-      <child link="camera_head_infra1_optical_frame" />
+      <parent link="${prefix}camera_head_infra1_frame" />
+      <child link="${prefix}camera_head_infra1_optical_frame" />
     </joint>
-    <link name="camera_head_infra1_optical_frame"/>
-    <joint name="camera_head_infra2_joint" type="fixed">
+    <link name="${prefix}camera_head_infra1_optical_frame"/>
+    <joint name="${prefix}camera_head_infra2_joint" type="fixed">
       <origin xyz="0 ${d435_cam_depth_to_infra2_offset} 0" rpy="0 0 0" />
-      <parent link="camera_head_link" />
-      <child link="camera_head_infra2_frame" />
+      <parent link="${prefix}camera_head_link" />
+      <child link="${prefix}camera_head_infra2_frame" />
     </joint>
-    <link name="camera_head_infra2_frame"/>
-    <joint name="camera_head_infra2_optical_joint" type="fixed">
+    <link name="${prefix}camera_head_infra2_frame"/>
+    <joint name="${prefix}camera_head_infra2_optical_joint" type="fixed">
       <origin xyz="0 0 0" rpy="${-M_PI/2} 0 ${-M_PI/2}" />
-      <parent link="camera_head_infra2_frame" />
-      <child link="camera_head_infra2_optical_frame" />
+      <parent link="${prefix}camera_head_infra2_frame" />
+      <child link="${prefix}camera_head_infra2_optical_frame" />
     </joint>
-    <link name="camera_head_infra2_optical_frame"/>
-    <joint name="camera_head_color_joint" type="fixed">
+    <link name="${prefix}camera_head_infra2_optical_frame"/>
+    <joint name="${prefix}camera_head_color_joint" type="fixed">
       <origin xyz="0 ${d435_cam_depth_to_color_offset} 0" rpy="0 0 0" />
-      <parent link="camera_head_link" />
-      <child link="camera_head_color_frame" />
+      <parent link="${prefix}camera_head_link" />
+      <child link="${prefix}camera_head_color_frame" />
     </joint>
-    <link name="camera_head_color_frame"/>
-    <joint name="camera_head_color_optical_joint" type="fixed">
+    <link name="${prefix}camera_head_color_frame"/>
+    <joint name="${prefix}camera_head_color_optical_joint" type="fixed">
       <origin xyz="0 0 0" rpy="${-M_PI/2} 0 ${-M_PI/2}" />
-      <parent link="camera_head_color_frame" />
-      <child link="camera_head_color_optical_frame" />
+      <parent link="${prefix}camera_head_color_frame" />
+      <child link="${prefix}camera_head_color_optical_frame" />
     </joint>
-    <link name="camera_head_color_optical_frame"/>
-<gazebo reference="camera_head_link">
-  <sensor name="camera_head" type="rgbd_camera">
+    <link name="${prefix}camera_head_color_optical_frame"/>
+<gazebo reference="${prefix}camera_head_link">
+  <sensor name="${prefix}camera_head" type="rgbd_camera">
     <camera>
       <horizontal_fov>1.5184</horizontal_fov>
@@ -158,5 +161,5 @@
          camera_head_depth_frame (zero rotation from camera_head_link)
          matches the data's true convention. -->
-    <gz_frame_id>camera_head_depth_frame</gz_frame_id>
+    <gz_frame_id>${prefix}camera_head_depth_frame</gz_frame_id>
     <output>
       <image>true</image>
@@ -168,3 +171,4 @@
 </gazebo>
   </xacro:if>
+  </xacro:macro>
 </robot>

File: ur_description/urdf/ur.urdf.xacro (robot description, xacro)
@@ -46,3 +46,4 @@
    <!-- Include Intel RealSense Camera -->
    <xacro:include filename="$(find ur_description)/urdf/intel_rgbd_cam_d435.urdf.xacro"/>
+   <xacro:intel_rgbd_cam_d435 prefix="$(arg tf_prefix)" parent_link="$(arg tf_prefix)base_link"/>
 </robot>
