Commit message: flatten pick table geometry

File: moveit_config/config/ur.srdf.xacro (robot description, xacro)
@@ -67,4 +67,15 @@
         <joint name="wrist_2_joint" value="0"/>
         <joint name="wrist_3_joint" value="1.0"/>
+    </group_state>
+    <!-- FK-screened joint-space via: tool0 ≈ (0.17, 0.00, 0.67), clear of
+         the pick-table AABB between base and object. -->
+    <group_state name="transit_clear" group="arm">
+        <!-- Rescreened: tool0≈(0.18,0.08,0.64), pan≈0 keeps gripper clear of torso. -->
+        <joint name="shoulder_pan_joint" value="-0.09"/>
+        <joint name="shoulder_lift_joint" value="-0.72"/>
+        <joint name="elbow_joint" value="-0.84"/>
+        <joint name="wrist_1_joint" value="-0.98"/>
+        <joint name="wrist_2_joint" value="1.79"/>
+        <joint name="wrist_3_joint" value="-0.04"/>
     </group_state>
     <group_state name="half_closed" group="gripper">
@@ -242,4 +253,15 @@
         <joint name="wrist_3_joint" value="1.0"/>
     </group_state>
+    <!-- FK-screened joint-space via: tool0 ≈ (0.17, 0.00, 0.67), clear of
+         the pick-table AABB between base and object. -->
+    <group_state name="transit_clear" group="arm">
+        <!-- Rescreened: tool0≈(0.18,0.08,0.64), pan≈0 keeps gripper clear of torso. -->
+        <joint name="shoulder_pan_joint" value="-0.09"/>
+        <joint name="shoulder_lift_joint" value="-0.72"/>
+        <joint name="elbow_joint" value="-0.84"/>
+        <joint name="wrist_1_joint" value="-0.98"/>
+        <joint name="wrist_2_joint" value="1.79"/>
+        <joint name="wrist_3_joint" value="-0.04"/>
+    </group_state>
     <group_state name="open" group="gripper">
         <joint name="gripper_joint" value="0.0"/>

File: moveit_config/config/ur_wrist_cam.srdf.xacro (robot description, xacro)
@@ -59,4 +59,15 @@
         <joint name="wrist_2_joint" value="0"/>
         <joint name="wrist_3_joint" value="1.0"/>
+    </group_state>
+    <!-- FK-screened joint-space via: tool0 ≈ (0.17, 0.00, 0.67), clear of
+         the pick-table AABB between base and object. -->
+    <group_state name="transit_clear" group="arm">
+        <!-- Rescreened: tool0≈(0.18,0.08,0.64), pan≈0 keeps gripper clear of torso. -->
+        <joint name="shoulder_pan_joint" value="-0.09"/>
+        <joint name="shoulder_lift_joint" value="-0.72"/>
+        <joint name="elbow_joint" value="-0.84"/>
+        <joint name="wrist_1_joint" value="-0.98"/>
+        <joint name="wrist_2_joint" value="1.79"/>
+        <joint name="wrist_3_joint" value="-0.04"/>
     </group_state>
     <group_state name="half_closed" group="gripper">
@@ -236,4 +247,15 @@
         <joint name="wrist_3_joint" value="1.0"/>
     </group_state>
+    <!-- FK-screened joint-space via: tool0 ≈ (0.17, 0.00, 0.67), clear of
+         the pick-table AABB between base and object. -->
+    <group_state name="transit_clear" group="arm">
+        <!-- Rescreened: tool0≈(0.18,0.08,0.64), pan≈0 keeps gripper clear of torso. -->
+        <joint name="shoulder_pan_joint" value="-0.09"/>
+        <joint name="shoulder_lift_joint" value="-0.72"/>
+        <joint name="elbow_joint" value="-0.84"/>
+        <joint name="wrist_1_joint" value="-0.98"/>
+        <joint name="wrist_2_joint" value="1.79"/>
+        <joint name="wrist_3_joint" value="-0.04"/>
+    </group_state>
     <group_state name="open" group="gripper">
         <joint name="gripper_joint" value="0.0"/>

Commit message: gripper fixes, RG2 default and README images

File: moveit_config/config/ur.srdf.xacro (robot description, xacro)
@@ -5,5 +5,5 @@
 -->
 <robot xmlns:xacro="http://www.ros.org/wiki/xacro" name="ur">
-    <xacro:arg name="gripper" default="robotiq_2f_85"/>
+    <xacro:arg name="gripper" default="$(optenv UR_GRIPPER onrobot_rg2)"/>
     <xacro:property name="selected_gripper" value="$(arg gripper)"/>
     <xacro:property name="gripper_base_link" value="${'robotiq_140_base_link' if selected_gripper == 'robotiq_2f_140' else 'robotiq_arg2f_base_link'}"/>

File: moveit_config/config/ur.urdf.xacro (robot description, xacro)
@@ -4,5 +4,5 @@
     <xacro:arg name="use_gazebo" default="true"/> <!-- Added missing argument -->
     <xacro:arg name="robot_name" default="ur"/>
-    <xacro:arg name="gripper" default="robotiq_2f_85"/>
+    <xacro:arg name="gripper" default="$(optenv UR_GRIPPER onrobot_rg2)"/>
     <xacro:arg name="name" default="ur"/>
     <xacro:arg name="ur_type" default="ur3"/>

File: moveit_config/config/ur_wrist_cam.srdf.xacro (robot description, xacro)
@@ -9,5 +9,5 @@
      otherwise register as a permanent self-collision. -->
 <robot xmlns:xacro="http://www.ros.org/wiki/xacro" name="ur">
-    <xacro:arg name="gripper" default="robotiq_2f_85"/>
+    <xacro:arg name="gripper" default="$(optenv UR_GRIPPER onrobot_rg2)"/>
     <xacro:property name="selected_gripper" value="$(arg gripper)"/>
     <xacro:property name="gripper_base_link" value="${'robotiq_140_base_link' if selected_gripper == 'robotiq_2f_140' else 'robotiq_arg2f_base_link'}"/>

File: moveit_config/config/ur_wrist_cam.urdf.xacro (robot description, xacro)
@@ -7,5 +7,5 @@
     <xacro:arg name="use_gazebo" default="true"/> <!-- Added missing argument -->
     <xacro:arg name="robot_name" default="ur"/>
-    <xacro:arg name="gripper" default="robotiq_2f_85"/>
+    <xacro:arg name="gripper" default="$(optenv UR_GRIPPER onrobot_rg2)"/>
     <xacro:arg name="name" default="ur"/>
     <xacro:arg name="ur_type" default="ur3"/>

File: robotiq_description/urdf/robotiq_2f_140.xacro (robot description, xacro)
@@ -130,4 +130,10 @@
   <xacro:macro name="inner_finger_pad" params="prefix fingerprefix">
     <link name="${prefix}${fingerprefix}_inner_finger_pad">
+      <!-- A link without inertia is lumped away / its collision ignored in the sim; give it a little mass. -->
+      <inertial>
+        <origin xyz="0 0 0" rpy="0 0 0" />
+        <mass value="0.005" />
+        <inertia ixx="1e-6" ixy="0" ixz="0" iyy="1e-6" iyz="0" izz="1e-6" />
+      </inertial>
       <visual>
         <origin xyz="0 0 0" rpy="0 0 0" />

File: ur_description/urdf/ur.urdf.xacro (robot description, xacro)
@@ -14,5 +14,5 @@
    <xacro:arg name="safety_k_position" default="20"/>
    <xacro:arg name="force_abs_paths" default="false"/>
-   <xacro:arg name="gripper" default="robotiq_2f_85"/>
+   <xacro:arg name="gripper" default="$(optenv UR_GRIPPER onrobot_rg2)"/>
    <xacro:arg name="robot_name" default="ur"/>
    <xacro:arg name="use_gazebo" default="true"/> <!-- Added missing argument -->

File: ur_description/urdf/ur_wrist_cam.urdf.xacro (robot description, xacro)
@@ -16,5 +16,5 @@
    <xacro:arg name="safety_k_position" default="20"/>
    <xacro:arg name="force_abs_paths" default="false"/>
-   <xacro:arg name="gripper" default="robotiq_2f_85"/>
+   <xacro:arg name="gripper" default="$(optenv UR_GRIPPER onrobot_rg2)"/>
    <xacro:arg name="robot_name" default="ur"/>
    <xacro:arg name="use_gazebo" default="true"/>

Commit message: MTC one-command launch, OnRobot gripper group fix

File: moveit_config/config/ur.srdf.xacro (robot description, xacro)
@@ -246,4 +246,17 @@
     <group name="gripper">
         <joint name="gripper_joint"/>
+        <!-- The mimic joints must be in the group too: MTC only lets the grasped object touch the links of
+             this group, so leaving the finger links out made every attached-object path "invalid" at execution. -->
+        <joint name="gripper_finger_1_truss_arm_joint"/>
+        <joint name="gripper_finger_1_finger_tip_joint"/>
+        <joint name="gripper_mirror_joint"/>
+        <joint name="gripper_finger_2_truss_arm_joint"/>
+        <joint name="gripper_finger_2_finger_tip_joint"/>
+        <!-- Fixed joints too: a link only belongs to the group if the joint above it is listed (the Robotiq
+             groups list their pad joints for the same reason). -->
+        <joint name="gripper_finger_1_origin_joint"/>
+        <joint name="gripper_finger_1_flex_finger_joint"/>
+        <joint name="gripper_finger_2_origin_joint"/>
+        <joint name="gripper_finger_2_flex_finger_joint"/>
     </group>
     <group name="arm_with_gripper">

File: moveit_config/config/ur_wrist_cam.srdf.xacro (robot description, xacro)
@@ -232,4 +232,17 @@
     <group name="gripper">
         <joint name="gripper_joint"/>
+        <!-- The mimic joints must be in the group too: MTC only lets the grasped object touch the links of
+             this group, so leaving the finger links out made every attached-object path "invalid" at execution. -->
+        <joint name="gripper_finger_1_truss_arm_joint"/>
+        <joint name="gripper_finger_1_finger_tip_joint"/>
+        <joint name="gripper_mirror_joint"/>
+        <joint name="gripper_finger_2_truss_arm_joint"/>
+        <joint name="gripper_finger_2_finger_tip_joint"/>
+        <!-- Fixed joints too: a link only belongs to the group if the joint above it is listed (the Robotiq
+             groups list their pad joints for the same reason). -->
+        <joint name="gripper_finger_1_origin_joint"/>
+        <joint name="gripper_finger_1_flex_finger_joint"/>
+        <joint name="gripper_finger_2_origin_joint"/>
+        <joint name="gripper_finger_2_flex_finger_joint"/>
     </group>
     <group name="arm_with_gripper">

Commit message: MTC final view-clear pose and slower approach

File: moveit_config/config/ur.srdf.xacro (robot description, xacro)
@@ -78,4 +78,14 @@
         <joint name="wrist_2_joint" value="1.79"/>
         <joint name="wrist_3_joint" value="-0.04"/>
+    </group_state>
+    <group_state name="view_clear" group="arm">
+        <!-- The simulator's start pose (initial_positions.yaml): the arm is out of the head camera's way, so the
+             point-cloud detector sees only the objects. MTC returns here after a place (arm_final_pose). -->
+        <joint name="shoulder_pan_joint" value="-0.1"/>
+        <joint name="shoulder_lift_joint" value="-1.6315"/>
+        <joint name="elbow_joint" value="0"/>
+        <joint name="wrist_1_joint" value="1.8251"/>
+        <joint name="wrist_2_joint" value="0"/>
+        <joint name="wrist_3_joint" value="1.2844"/>
     </group_state>
     <group_state name="half_closed" group="gripper">
@@ -291,4 +301,14 @@
         <joint name="wrist_3_joint" value="-0.04"/>
     </group_state>
+    <group_state name="view_clear" group="arm">
+        <!-- The simulator's start pose (initial_positions.yaml): the arm is out of the head camera's way, so the
+             point-cloud detector sees only the objects. MTC returns here after a place (arm_final_pose). -->
+        <joint name="shoulder_pan_joint" value="-0.1"/>
+        <joint name="shoulder_lift_joint" value="-1.6315"/>
+        <joint name="elbow_joint" value="0"/>
+        <joint name="wrist_1_joint" value="1.8251"/>
+        <joint name="wrist_2_joint" value="0"/>
+        <joint name="wrist_3_joint" value="1.2844"/>
+    </group_state>
     <group_state name="open" group="gripper">
         <joint name="gripper_joint" value="0.0"/>

File: moveit_config/config/ur_wrist_cam.srdf.xacro (robot description, xacro)
@@ -70,4 +70,14 @@
         <joint name="wrist_2_joint" value="1.79"/>
         <joint name="wrist_3_joint" value="-0.04"/>
+    </group_state>
+    <group_state name="view_clear" group="arm">
+        <!-- The simulator's start pose (initial_positions.yaml): the arm is out of the head camera's way, so the
+             point-cloud detector sees only the objects. MTC returns here after a place (arm_final_pose). -->
+        <joint name="shoulder_pan_joint" value="-0.1"/>
+        <joint name="shoulder_lift_joint" value="-1.6315"/>
+        <joint name="elbow_joint" value="0"/>
+        <joint name="wrist_1_joint" value="1.8251"/>
+        <joint name="wrist_2_joint" value="0"/>
+        <joint name="wrist_3_joint" value="1.2844"/>
     </group_state>
     <group_state name="half_closed" group="gripper">
@@ -277,4 +287,14 @@
         <joint name="wrist_3_joint" value="-0.04"/>
     </group_state>
+    <group_state name="view_clear" group="arm">
+        <!-- The simulator's start pose (initial_positions.yaml): the arm is out of the head camera's way, so the
+             point-cloud detector sees only the objects. MTC returns here after a place (arm_final_pose). -->
+        <joint name="shoulder_pan_joint" value="-0.1"/>
+        <joint name="shoulder_lift_joint" value="-1.6315"/>
+        <joint name="elbow_joint" value="0"/>
+        <joint name="wrist_1_joint" value="1.8251"/>
+        <joint name="wrist_2_joint" value="0"/>
+        <joint name="wrist_3_joint" value="1.2844"/>
+    </group_state>
     <group_state name="open" group="gripper">
         <joint name="gripper_joint" value="0.0"/>
