Commit message: switch to bullet physics, fix gripper mount offsets

File: ur_description/urdf/ur_macro.xacro (robot description, xacro)
@@ -343,5 +343,5 @@
       <parent link="${tf_prefix}tool0"/>
       <child link="${tf_prefix}robotiq_arg2f_base_link"/>
-      <origin xyz="0 0 0.005" rpy="0 0 0"/>
+      <origin xyz="0 0 0.01" rpy="0 0 0"/>
       <gazebo><disableFixedJointLumping>true</disableFixedJointLumping></gazebo>
     </joint>
@@ -350,5 +350,5 @@
   <xacro:if value="${gripper == 'robotiq_2f_140'}">
     <xacro:robotiq_gripper name="robotiq_140" prefix="" parent="${tf_prefix}tool0" include_ros2_control="false">
-      <origin xyz="0 0 0.005" rpy="0 0 0"/>
+      <origin xyz="0 0 0.01" rpy="0 0 0"/>
     </xacro:robotiq_gripper>
   </xacro:if>
