Commit message: fix grasp height, close width, pad friction and place pose

File: robotiq_2f_85_gripper_visualization/urdf/robotiq_arg2f_85_model_macro.xacro (robot description, xacro)
@@ -120,4 +120,9 @@
       </collision>
     </link>
+    <!-- Grippy rubber pads: unset friction fell back to the simulator default and the cube slipped out -->
+    <gazebo reference="${prefix}${fingerprefix}_inner_finger_pad">
+      <mu1>2.0</mu1>
+      <mu2>2.0</mu2>
+    </gazebo>
   </xacro:macro>
   <xacro:macro name="outer_finger_joint" params="prefix fingerprefix">

File: ur_description/urdf/intel_rgbd_cam_d435_wrist.urdf.xacro (robot description, xacro)
@@ -16,12 +16,20 @@
          gripper body, tilt/yaw re-aim it at the TCP so the fingers don't
          block the center of frame. Starting guess only - verify in RViz. -->
-    <xacro:property name="wrist_cam_offset_y" value="0.055"/>
-    <xacro:property name="wrist_cam_offset_z" value="-0.02"/>
+    <!-- The gz camera looks along its link +X. The pitch of -90 deg turns that
+         onto tool0 +Z (out along the fingers); the tilt then leans it a further
+         wrist_cam_tilt_deg, and the 180 deg yaw about tool0 Z makes that lean
+         point at the gripper axis (-X, since the camera sits at +X). To move
+         the camera to the other side use offset_x=-0.065 with yaw 0, or offset_y
+         with yaw -90 / +90. The old yaw of -15 left the camera leaning along +X, and
+         with z=-0.02 it sat behind the flange and mostly saw the wrist housing. -->
+    <xacro:property name="wrist_cam_offset_x" value="0.065"/>
+    <xacro:property name="wrist_cam_offset_y" value="0.0"/>
+    <xacro:property name="wrist_cam_offset_z" value="0.0"/>
     <xacro:property name="wrist_cam_tilt_deg" value="20"/>
-    <xacro:property name="wrist_cam_yaw_deg" value="-15"/>
+    <xacro:property name="wrist_cam_yaw_deg" value="180"/>
     <joint name="$(arg prefix)tool0_to_camera_wrist_link" type="fixed">
       <parent link="$(arg prefix)tool0"/>
       <child link="camera_wrist_link" />
-      <origin xyz="0 ${wrist_cam_offset_y} ${wrist_cam_offset_z}"
+      <origin xyz="${wrist_cam_offset_x} ${wrist_cam_offset_y} ${wrist_cam_offset_z}"
               rpy="0.0 ${-M_PI/2 + wrist_cam_tilt_deg * M_PI / 180} ${wrist_cam_yaw_deg * M_PI / 180}"/>
       <!-- Without this, SDFormat lumps this fixed joint's link into
